Commit message: Make the contact-priority pipeline the mainline solver
The previous merge kept the foot-orientation solver as the base and landed only
the standalone contact modules, so the lexicographic end-effector solver that
produced the good c167 result was not actually running. Reverse that: the
contact-priority line is now the mainline pipeline.

core.py, retargeting.py, main.py and utils.py come from 7033d12 unchanged, so
the solver, the trajectory refinement pass and the CLI behave exactly as they
did at the end of yesterday's session.

Kept from the foot-orientation line, because it is additive rather than a
competing solver:

- omniretargeting/data_sources/ — the LAFAN1, NOKOV, OMOMO, BVH and SMPL-X
  adapters plus the registry, with tests/data_sources and config_templates/.
- robot_models/booster_k1/ and robot_models/hightorque_mini_pi_plus/.
- visualizer.py, filter.py, batch.py, docs/ADDING_SOURCE_ADAPTERS.md, agents/.

The adapters needed interpolation, body-height and floating-base URDF helpers
that only existed in the other utils.py, so those 14 functions are ported over.
They are additive; nothing in the contact-priority code is redefined.
create_flat_terrain is deliberately not ported, since main.py already has it.

Dropped, as the solver they belong to is no longer mainline: foot_frames.py,
scene_contact.py, the two diagnostic scripts that import them, and the ten test
modules covering that solver. All of it stays reachable at 3822b3f.

Tests: 87 passed, 4 failed, 4 skipped. The 4 failures are the g1/h1 mesh-path
errors that this branch's URDF has always had -- identical to 7033d12 on its
own -- not a regression from the assembly.

Verified end to end on test_data/c167_1530_final_v3: contact inference, the
staged solve and the 16-step refinement all run, and the output carries the
same 15 keys, joint_names and contact_names as yesterday's artefacts. Scene
penetration lands at 4.12 cm max, 1.67 cm mean, 14 of 144 frames, under the
10 cm bar in AGENTS.md.

Co-Authored-By: Claude Opus 5 <noreply@anthropic.com>

File: robot_models/unitree_g1/g1_29dof_popsicle.urdf (robot description, URDF)
Before this commit: robot g1, 40 links, 39 joints
Links:
- added link world
Joints:
- added joint floating_base_joint: type floating, parent world, child pelvis

File: robot_models/unitree_h1/h1.urdf (robot description, URDF)
Before this commit: robot h1_description, 25 links, 24 joints
Links:
- added link world
Joints:
- added joint floating_base_joint: type floating, parent world, child pelvis
